File: lora-bluepill-sch.kicad_pcb (KiCad board)
At the start: 2 copper layers, 70 x 55 mm, 37 parts, among them J1 Conn_01x04_Male, J2 Conn_01x04_Female, J3 Conn_01x07_Female, J4 Conn_01x10_Male, U1 RadioEnge_LoRaWAN, U2 YAAJ_BluePill, U3 FTDI_Breakout, U4 LM35-LP, U5 L293D

Commit message: Version sent to Fabrication
Parts:
- added FID1: Fiducial, Project Footprints:labsc-logo, B.Cu at (62.5, 93.5)
Connections:
- J4 pad 2: unconnected-(J4-Pad2) -> GND
- J4 pad 8: unconnected-(J4-Pad8) -> GND
- J4 pad 9: unconnected-(J4-Pad9) -> GND
Other:
- board text added: "12V"
- board text added: "3V3"
- board text added: "5V"
- board text added: "Bluepill"
- board text added: "Dez/2022"
- board text added: "FTDI 5V"
- board text added: "GND"
- board text added: "L1_N"
- board text added: "L1_P"
- board text added: "L2_N"
- board text added: "L2_P"
- board text added: "LED1"
- board text added: "LED4"
- board text added: "LM35+L293"
- board text added: "PB3"
- board text added: "PB4"
- board text added: "PB5"
- board text added: "PB8"
- board text added: "PB9"
- board text added: "RX"
- board text added: "TX"
