File: lora-bluepill-sch.kicad_pcb (KiCad board)
At the start: 2 copper layers, 70 x 55 mm, 38 parts, among them J1 Conn_01x04_Male, J2 Conn_01x04_Female, J3 Conn_01x07_Female, J4 Conn_01x10_Male, U1 RadioEnge_LoRaWAN, U2 YAAJ_BluePill, U3 FTDI_Breakout, U4 LM35-LP, U5 L293D

Commit message: add footprints, wip
Co-Authored-By: Claude Sonnet 5 <noreply@anthropic.com>
Parts:
- added C1: 100n, Capacitor_THT:C_Disc_D6.0mm_W4.4mm_P5.00mm, F.Cu at (220.0, 42.9)
- added C10: 10u, Capacitor_SMD:CP_Elec_5x3, F.Cu at (188.2, 97.9)
- added C11: 100n, Capacitor_THT:C_Disc_D6.0mm_W4.4mm_P5.00mm, F.Cu at (220.0, 66.7)
- added C12: 2.2u, Capacitor_SMD:CP_Elec_4x3, F.Cu at (221.6, 99.3)
- added C2: 100n, Capacitor_THT:C_Disc_D6.0mm_W4.4mm_P5.00mm, F.Cu at (220.0, 48.8)
- added C3: 100n, Capacitor_THT:C_Disc_D6.0mm_W4.4mm_P5.00mm, F.Cu at (220.0, 54.8)
- added C7: 100n, Capacitor_THT:C_Disc_D6.0mm_W4.4mm_P5.00mm, F.Cu at (220.0, 60.7)
- added M1: ~, LabSC:ESP32C6-Minimal, F.Cu at (149.5, 47.5)
- added M2: ~, LabSC:Waveshare-LR1121, F.Cu at (164.1, 20.0)
- added M3: ~, LabSC:A1205S-2W, F.Cu at (207.9, 104.4)
- added Q1: BC558, Package_TO_SOT_THT:TO-92_Inline, F.Cu at (219.3, 76.4)
- added R10: 1K, Resistor_THT:R_Axial_DIN0204_L3.6mm_D1.6mm_P7.62mm_Horizontal, F.Cu at (209.3, 50.9)
- added R11: 1K, Resistor_THT:R_Axial_DIN0204_L3.6mm_D1.6mm_P7.62mm_Horizontal, F.Cu at (209.3, 54.1)
- added R12: 1K, Resistor_THT:R_Axial_DIN0204_L3.6mm_D1.6mm_P7.62mm_Horizontal, F.Cu at (209.3, 57.2)
- added R13: 100R, Resistor_THT:R_Axial_DIN0204_L3.6mm_D1.6mm_P7.62mm_Horizontal, F.Cu at (209.3, 60.4)
- added R14: 82K, Resistor_THT:R_Axial_DIN0204_L3.6mm_D1.6mm_P7.62mm_Horizontal, F.Cu at (209.3, 63.5)
- added R15: 1K, Resistor_THT:R_Axial_DIN0204_L3.6mm_D1.6mm_P7.62mm_Horizontal, F.Cu at (209.3, 66.7)
- added R16: 1K, Resistor_THT:R_Axial_DIN0204_L3.6mm_D1.6mm_P7.62mm_Horizontal, F.Cu at (209.3, 69.8)
- added R7: 1K, Resistor_THT:R_Axial_DIN0204_L3.6mm_D1.6mm_P7.62mm_Horizontal, F.Cu at (209.3, 41.5)
- added R8: 1K, Resistor_THT:R_Axial_DIN0204_L3.6mm_D1.6mm_P7.62mm_Horizontal, F.Cu at (209.3, 44.6)
- added R9: 1K, Resistor_THT:R_Axial_DIN0204_L3.6mm_D1.6mm_P7.62mm_Horizontal, F.Cu at (209.3, 47.8)
- added U1: YAAJ_BlackPill, Footprints:YAAJ_WeAct_BlackPill_2, F.Cu at (154.4, 93.1)
- added U4: PC817, Package_DIP:DIP-4_W7.62mm, F.Cu at (198.6, 42.0)
- added U5: PC817, Package_DIP:DIP-4_W7.62mm, F.Cu at (198.6, 48.6)
- added U6: PC817, Package_DIP:DIP-4_W7.62mm, F.Cu at (198.6, 55.2)
- added U7: PC817, Package_DIP:DIP-4_W7.62mm, F.Cu at (198.6, 61.9)
- added U8: PC817, Package_DIP:DIP-4_W7.62mm, F.Cu at (198.6, 68.5)
- added U9: NE555P, Package_DIP:DIP-8_W7.62mm, F.Cu at (243.4, 74.4)
- renumbered C1 to C4, C2 to C5, C3 to C6, C4 to C8, C5 to C9, D6 to D1, D8 to D2, D7 to D3, D1 to D4, D3 to D5, D5 to D6, D2 to D7, D4 to D8, J1 to J4, R4 to R1, R6 to R2, R1 to R3, R5 to R4, R3 to R5, R2 to R6, U3 to U2, U1 to U3
Connections:
- D4 pad 1: /STM_TX -> /UART_AT_TX
- D5 pad 1: /STM_RX -> /UART_AT_RX
- D7 pad 1: /STM_TX -> /UART_AT_TX
- R1 pad 2: /PA3 -> /LED1
- R2 pad 2: /PA5 -> /LED2
- R4 pad 2: /PA2 -> /LED3
- R5 pad 2: /PA4 -> /LED4

Commit message: WIP: schematic/PCB progress, screw terminals, ESP32-C6 reference
Design work in progress on the LoRa carrier:
  - schematic and PCB updates
  - HANDSON KF301-2P / KF301-4P screw terminal footprints
  - Custom_Symbols.kicad_sym
  - Connector.kicad_sym additions, fp-lib-table / sym-lib-table updates
  - Waveshare-LR1121 footprint tweak
  - nanoESP32C6.pdf: module reference schematic. Confirms the onboard LED is
    an addressable RGB (WS2812-type) driven from GPIO8, not a plain GPIO LED.

Bumps the Kicad-STM32 submodule to 244753d, which adds the two BlackPill
symbols that were sitting untracked in the submodule working tree.

Co-Authored-By: Claude Opus 4.8 <noreply@anthropic.com>
Parts:
- removed the C6 at (110.7, 96.2)
- removed the C8 at (86.9, 72.4)
- removed the C9 at (61.3, 61.2)
- removed J3: Conn_01x07_Female, Connector_PinSocket_2.54mm:PinSocket_1x07_P2.54mm_Vertical
- removed the J4 at (87.9, 104.6)
- removed the R7 at (109.6, 86.2)
- removed the R8 at (109.2, 72.4)
- removed U1: YAAJ_BlackPill, Footprints:YAAJ_WeAct_BlackPill_2
- removed the U2 at (67.5, 76.2)
- removed the U4 at (110.8, 100.6)
- removed the U5 at (82.9, 64.8)
- added J1: Conn_01x05, Connector_PinHeader_2.54mm:PinHeader_1x05_P2.54mm_Horizontal, F.Cu at (178.6, -2.83)
- added J10: Screw_Terminal_01x04, KF301-2P:HANDSON_KF301-4P, F.Cu at (180.1, 14.4)
- added J11: Screw_Terminal_01x04, KF301-2P:HANDSON_KF301-4P, F.Cu at (180.1, 23.4)
- added J5: Conn_01x02, Connector_PinHeader_2.54mm:PinHeader_1x02_P2.54mm_Vertical, F.Cu at (212.7, 11.9)
- added J7: Screw_Terminal_01x02, KF301-2P:HANDSON_KF301-2P, F.Cu at (204.7, 14.4)
- added J8: Screw_Terminal_01x02, KF301-2P:HANDSON_KF301-2P, F.Cu at (204.7, 23.4)
- added U10: YAAJ_WeAct_BlackPill_Part_Like, Footprints:YAAJ_WeAct_BlackPill_2, F.Cu at (41.8, 50.7)
- C10: footprint Capacitor_SMD:CP_Elec_5x3 -> Capacitor_THT:CP_Radial_D5.0mm_P2.50mm
- C12: footprint Capacitor_SMD:CP_Elec_4x3 -> Capacitor_THT:CP_Radial_D5.0mm_P2.50mm
- J2: value Conn_01x04_Female -> Conn_01x05; footprint Connector_PinSocket_2.54mm:PinSocket_1x04_P2.54mm_Vertical -> Connector_PinHeader_2.54mm:PinHeader_1x05_P2.54mm_Horizontal
- moved M2 124.2 mm to (42.8, 46.6), turned to 0 degrees
- moved J2 113.5 mm to (191.9, -2.83), turned to 0 degrees
- moved M1 106.5 mm to (43.2, 41.1), turned to 180 degrees
- moved U3 63.3 mm to (30.9, 50.0)
Connections:
- J2 pad 1: +3V3 -> /MISO
- J2 pad 2: GND -> /TEMP1_SSEL
- J2 pad 3: /I2C1_SCL -> /SCLK
- J2 pad 4: /I2C1_SDA -> +3V3
- M1 pad 10: /IN2_3V3 -> unconnected-(M1-D8-Pad10)
- M1 pad 11: /LR1121_SSEL -> /LR1121_BUSY
- M1 pad 12: /LR1121_RESET -> /LR1121_IRQ
- M1 pad 18: /OUT2_3V3 -> unconnected-(M1-D9-Pad18)
- M1 pad 19: /LR1121_BUSY -> unconnected-(M1-D18-Pad19)
- M1 pad 20: /TEMP1_SSEL -> /IN2_3V3
- M1 pad 21: /TEMP2_SSEL -> /OUT1_3V3
- M1 pad 23: /LED3 -> unconnected-(M1-D22-Pad23)
- M1 pad 25: /LED4 -> /OUT2_3V3
- M1 pad 26: /UART_AT_TX -> /UART_AT_RX
- M1 pad 27: /UART_AT_RX -> /UART_AT_TX
- M1 pad 28: /LR1121_IRQ -> unconnected-(M1-D3-Pad28)
- M1 pad 29: /MISO -> unconnected-(M1-D2-Pad29)
- M1 pad 4: unconnected-(M1-D4-Pad4) -> /TEMP1_SSEL
- M1 pad 5: /TEMP3_SSEL -> /LR1121_SSEL
- M1 pad 7: /MOSI -> /MISO
- M1 pad 8: /LED1 -> /MOSI
- M1 pad 9: /LED2 -> /LR1121_RESET
Routing:
- net +3V3: track 193.5 -> 0.00 mm, vias 5 -> 0
- net +5V_LM35: track 131.4 -> 0.00 mm, vias 3 -> 0
- net +5V: track 55.0 -> 0.00 mm, vias 2 -> 0
- net /ADC1_IN1: track 50.2 -> 0.00 mm, vias 2 -> 0
- net /STM_RX: track 38.5 -> 0.00 mm, vias 1 -> 0
- net /PB8: track 34.9 -> 0.00 mm, vias 2 -> 0
- net /PB9: track 33.3 -> 0.00 mm, vias 2 -> 0
- net /PB5: track 29.6 -> 0.00 mm
- net /PB3: track 29.5 -> 0.00 mm
- net /PB4: track 29.4 -> 0.00 mm
- net /L1_P: track 26.6 -> 0.00 mm, vias 1 -> 0
- net /L2_N: track 26.2 -> 0.00 mm, vias 1 -> 0
- net /I2C1_SCL: track 21.7 -> 0.00 mm, vias 1 -> 0
- net /PB0: track 20.3 -> 0.00 mm, vias 1 -> 0
- net /I2C1_SDA: track 20.3 -> 0.00 mm, vias 1 -> 0
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- removed copper zone on B.Cu, net GND
- removed copper zone on F.Cu, net GND
Other:
- board size 70 x 55 mm -> 70 x 70 mm
