File: lora-bluepill-sch.kicad_pcb (KiCad board)
At the start: 2 copper layers, 70 x 70 mm, 62 parts, among them J1 Conn_01x05, J10 Screw_Terminal_01x04, J11 Screw_Terminal_01x04, J2 Conn_01x05, J4 Conn_01x04_Male, J5 Conn_01x02, J7 Screw_Terminal_01x02, J8 Screw_Terminal_01x02, Q1 BC558, U10 YAAJ_WeAct_BlackPill_Part_Like, U2 FTDI_Breakout, U3 RadioEnge_LoRaWAN, U4 PC817, U5 PC817, U6 PC817, U7 PC817, U8 PC817, U9 NE555P

Commit message: placement evolution
Parts:
- added R17: 1K, Resistor_THT:R_Axial_DIN0204_L3.6mm_D1.6mm_P7.62mm_Horizontal, F.Cu at (40.7, 46.8)
- moved J2 160.8 mm to (32.5, 18.1), turned to 90 degrees
- moved U9 159.5 mm to (84.7, 58.9), turned to 0 degrees
- moved C7 156.9 mm to (64.0, 78.0), turned to -90 degrees
- moved C3 155.1 mm to (65.5, 68.2), turned to 90 degrees
- moved C12 154.2 mm to (87.2, 23.7), turned to 180 degrees
- moved R10 152.8 mm to (57.0, 38.4), turned to -90 degrees
- moved M3 147.8 mm to (87.2, 19.2)
- moved C2 146.3 mm to (78.5, 86.0)
- moved R12 145.8 mm to (63.8, 48.7), turned to 180 degrees
- moved R7 145.7 mm to (64.3, 56.2), turned to 180 degrees
- moved R9 145.1 mm to (65.0, 32.2), turned to -90 degrees
- moved R11 145.1 mm to (64.3, 58.7), turned to 180 degrees
- moved C1 140.1 mm to (84.0, 76.5)
- moved Q1 140.0 mm to (79.8, 65.8), turned to 180 degrees
- moved C10 138.9 mm to (71.0, 23.2), turned to 180 degrees
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Connections:
- net /AT_RX renamed Net-(D7-A)
- M1 pad 20: /IN2_3V3 -> unconnected-(M1-D19-Pad20)
- M1 pad 23: unconnected-(M1-D22-Pad23) -> /UART_AT_TX
- M1 pad 24: /IN1_3V3 -> /UART_AT_RX
- M1 pad 26: /UART_AT_RX -> /IN2_3V3
- M1 pad 27: /UART_AT_TX -> unconnected-(M1-TX-Pad27)
- M1 pad 28: unconnected-(M1-D3-Pad28) -> /IN1_3V3
- M1 pad 29: unconnected-(M1-D2-Pad29) -> /TEMP2_SSEL
- U10 pad 26: unconnected-(U10-PA0-Pad26) -> /OUT1_3V3
- U10 pad 27: unconnected-(U10-PA1-Pad27) -> /LM555_ON_PULSE
- U10 pad 30: /IN2_3V3 -> /OUT2_3V3
- U10 pad 31: unconnected-(U10-PA5-Pad31) -> /IN2_3V3
- U10 pad 32: /OUT2_3V3 -> unconnected-(U10-PA6-Pad32)
- U10 pad 35: /LM555_ON_PULSE -> unconnected-(U10-PB1-Pad35)
- U10 pad 37: /OUT1_3V3 -> unconnected-(U10-PB10-Pad37)
- U3 pad 3: /STM_RX -> /UART_AT_RX
Other:
- board size 70 x 70 mm -> 100 x 80 mm
- board text removed: "12V"
- board text removed: "3V3"
- board text removed: "5V"
- board text removed: "Bluepill"
- board text removed: "FTDI 5V"
- board text removed: "GND"
- board text removed: "L1_N"
- board text removed: "L1_P"
- board text removed: "L2_N"
- board text removed: "L2_P"
- board text removed: "LED4"
- board text removed: "LM35+L293"
- board text removed: "PB3"
- board text removed: "PB4"
- board text removed: "PB5"
- board text removed: "PB8"
- board text removed: "PB9"
- board text removed: "RX"
- board text removed: "TX"

Commit message: board finished, but not checked
Parts:
- removed C7, C8: 100n, Capacitor_THT:C_Disc_D6.0mm_W4.4mm_P5.00mm
- removed J4: Conn_01x04_Male, Connector_PinSocket_2.54mm:PinSocket_1x04_P2.54mm_Vertical
- added C13: 100n, Capacitor_THT:C_Disc_D6.0mm_W4.4mm_P5.00mm, F.Cu at (68.6, 14.9)
- added C14: 100n, Capacitor_THT:C_Disc_D6.0mm_W4.4mm_P5.00mm, F.Cu at (6.35, 64.7)
- added C15: 100n, Capacitor_THT:C_Disc_D6.0mm_W4.4mm_P5.00mm, F.Cu at (94.0, 48.3)
- added C16: 100n, Capacitor_THT:C_Disc_D6.0mm_W4.4mm_P5.00mm, F.Cu at (81.3, 12.7)
- moved C6 66.1 mm to (52.3, 18.6), turned to 90 degrees
- moved C9 65.6 mm to (16.3, 22.9), turned to -90 degrees
- moved C3 58.7 mm to (24.4, 26.3)
- moved C2 55.4 mm to (27.7, 64.0), turned to -90 degrees
- moved R15 35.1 mm to (88.9, 7.62)
- moved C1 33.3 mm to (53.3, 63.5), turned to -90 degrees
- moved C11 31.9 mm to (88.8, 68.6), turned to 180 degrees
- moved R14 31.7 mm to (82.3, 62.0), turned to 0 degrees
- moved C4 27.3 mm to (36.8, 55.9), turned to -90 degrees
- moved J10 25.6 mm to (95.5, 55.0), turned to -90 degrees
- moved R17 23.6 mm to (63.5, 40.6), turned to 180 degrees
- moved H3 23.1 mm to (85.0, 5.00)
- moved R13 22.6 mm to (89.9, 59.7), turned to 180 degrees
- moved R16 17.3 mm to (88.9, 19.1)
- moved U3 16.7 mm to (20.3, 33.0)
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Connections:
- net /FTDI_RX renamed Net-(D4-A)
- J10 pad 1: /OUT1_OC -> HI_GND
- J10 pad 2: HI_GND -> /OUT2_OC
- J10 pad 3: /OUT2_OC -> HI_GND
- J10 pad 4: HI_GND -> /OUT1_OC
- M1 pad 18: unconnected-(M1-D9-Pad18) -> /EXP_C6_TX
- M1 pad 19: unconnected-(M1-D18-Pad19) -> /EXP_C6_SCL
- M1 pad 20: unconnected-(M1-D19-Pad20) -> /EXP_C6_SDA
- M1 pad 23: /UART_AT_TX -> /EXP_C6_RX
- M1 pad 24: /UART_AT_RX -> /IN2_3V3
- M1 pad 26: /IN2_3V3 -> /UART_AT_RX
- M1 pad 27: unconnected-(M1-TX-Pad27) -> /UART_AT_TX
- U10 pad 5: unconnected-(U10-PA8-Pad5) -> /TEMP1_SSEL
- U10 pad 9: /TEMP1_SSEL -> unconnected-(U10-PA12-Pad9)
- U2 pad 4: /FTDI_5V -> unconnected-(U2-VCC-Pad4)
Routing:
- net GND: track 0.00 -> 348.4 mm, vias 0 -> 8
- net +3V3: track 0.00 -> 262.5 mm, vias 0 -> 8
- net HI_GND: track 0.00 -> 189.2 mm, vias 0 -> 3
- net +5V: track 0.00 -> 131.2 mm, vias 0 -> 2
- net /MISO: track 0.00 -> 97.0 mm, vias 0 -> 3
- net +12V: track 0.00 -> 90.6 mm
- net /SCLK: track 0.00 -> 83.1 mm, vias 0 -> 3
- net /UART_AT_RX: track 0.00 -> 49.9 mm, vias 0 -> 1
- net Net-(D7-A): track 0.00 -> 42.7 mm, vias 0 -> 1
- net /TEMP1_SSEL: track 0.00 -> 38.0 mm, vias 0 -> 2
- net /OUT2_OC: track 0.00 -> 34.8 mm, vias 0 -> 1
- net /UART_AT_TX: track 0.00 -> 34.5 mm, vias 0 -> 1
- net /LR1121_IRQ: track 0.00 -> 33.7 mm, vias 0 -> 1
- net /MOSI: track 0.00 -> 33.4 mm, vias 0 -> 2
- net Net-(D4-A): track 0.00 -> 31.8 mm
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- added copper zone on B.Cu, net GND
- added copper zone on F.Cu, net GND
- added copper zone on B.Cu, net HI_GND
- added copper zone on F.Cu, net HI_GND
Other:
- board text removed: "LED1"
