File: lora-bluepill-sch.kicad_sch (KiCad schematic)
At the start: 38 parts, among them J1 Conn_01x04_Male, J2 Conn_01x04_Female, J3 Conn_01x07_Female, J4 Conn_01x10_Male, U1 RadioEnge_LoRaWAN, U2 YAAJ_BluePill, U3 FTDI_Breakout, U4 LM35-LP, U5 L293D

Commit message: Version sent to Fabrication
Parts:
- FID1: renamed from FID?; footprint (none) -> Project Footprints:labsc-logo
Connections:
- net GND: now also J4.2 (Pin_2), J4.8 (Pin_8), J4.9 (Pin_9)
Other:
- moved on the sheet: D5, D6, D7, D8, J4, R3, R4, R5, R6
