File: lora-bluepill-sch.kicad_sch (KiCad schematic)
At the start: 38 parts, among them J1 Conn_01x04_Male, J2 Conn_01x04_Female, J3 Conn_01x07_Female, J4 Conn_01x10_Male, U1 RadioEnge_LoRaWAN, U2 YAAJ_BluePill, U3 FTDI_Breakout, U4 LM35-LP, U5 L293D

Commit message: Continue design work: WeAct BlackPill footprint, screw connectors
Vendor YAAJ_WeAct_BlackPill_2 footprint locally (was pulled in via
Kicad-STM32 submodule path) to keep the project self-contained, and
add the Screw01x02/Screw01x04 connectors used for the new module
variant. Includes accompanying schematic/PCB/project updates.

Co-Authored-By: Claude Sonnet 5 <noreply@anthropic.com>
Parts:
- removed C6, C8: 100n, Capacitor_THT:C_Disc_D6.0mm_W4.4mm_P5.00mm, symbol Device:C
- removed C9: 10uF / 25V, Capacitor_THT:CP_Radial_D5.0mm_P2.50mm, symbol Device:C_Polarized_US
- removed J2: Conn_01x04_Female, Connector_PinSocket_2.54mm:PinSocket_1x04_P2.54mm_Vertical, symbol Connector:Conn_01x04_Female
- removed J3: Conn_01x07_Female, Connector_PinSocket_2.54mm:PinSocket_1x07_P2.54mm_Vertical, symbol Connector:Conn_01x07_Female
- removed J4: Conn_01x10_Male, Connector_PinSocket_2.54mm:PinSocket_1x10_P2.54mm_Vertical, symbol Connector:Conn_01x10_Male
- removed U2: YAAJ_BluePill, Footprints:YAAJ_BluePill_2, symbol YAAJ_BluePill:YAAJ_BluePill
- removed U4: LM35-LP, Connector_PinSocket_2.54mm:PinSocket_1x03_P2.54mm_Vertical, symbol Sensor_Temperature:LM35-LP
- removed U5: L293D, Package_DIP:DIP-16_W7.62mm, symbol Driver_Motor:L293D
- added C1, C11, C2, C3, C7: 100n, Capacitor_THT:C_Disc_D6.0mm_W4.4mm_P5.00mm, symbol Device:C
- added C10: 10u, Capacitor_SMD:CP_Elec_5x3, symbol Device:C
- added C12: 2.2u, Capacitor_SMD:CP_Elec_4x3, symbol Device:C
- added J1, J2, J3: Conn_01x05, symbol Connector_Generic:Conn_01x05
- added J5: Conn_01x02, symbol Connector_Generic:Conn_01x02
- added J6, J9: (no value), symbol Connector:Screw01x02
- added J7, J8: (no value), symbol Connector:Screw01x04
- added M1: (no value), symbol LabSC:ESP32C6Minimal
- added M2: (no value), symbol LabSC:LR1121-WAVESHARE-Core1121
- added M3: (no value), symbol power:A1205S-2WR3
- added Q1: BC558, Package_TO_SOT_THT:TO-92_Inline, symbol Transistor_BJT:BC558
- added R10, R11, R12, R15, R16, R9: 1K, Resistor_THT:R_Axial_DIN0204_L3.6mm_D1.6mm_P7.62mm_Horizontal, symbol Device:R
- added R13: 100R, Resistor_THT:R_Axial_DIN0204_L3.6mm_D1.6mm_P7.62mm_Horizontal, symbol Device:R
- added R14: 82K, Resistor_THT:R_Axial_DIN0204_L3.6mm_D1.6mm_P7.62mm_Horizontal, symbol Device:R
- added U1: YAAJ_BlackPill, Footprints:YAAJ_WeAct_BlackPill_2, symbol YAAJ_BlackPill:YAAJ_BlackPill
- added U4, U5, U6, U7, U8: PC817, Package_DIP:DIP-4_W7.62mm, symbol Isolator:PC817
- added U9: NE555P, Package_DIP:DIP-8_W7.62mm, symbol Timer:NE555P
- R7, R8: value 10k -> 1K
- renumbered C1 to C4, C2 to C5, C3 to C6, C4 to C8, C5 to C9, D6 to D1, D8 to D2, D7 to D3, D1 to D4, D3 to D5, D5 to D6, D2 to D7, D4 to D8, J1 to J4, R4 to R1, R6 to R2, R1 to R3, R5 to R4, R3 to R5, R2 to R6, U3 to U2, U1 to U3
Connections:
- net +12V: now also R8.2, C12.1, J6.1, M3.1 (VIN), R14.2, R15.1, R16.1, U9.8 (VCC)
- net +3V3: now also C3.1, C7.1, J1.4 (Pin_4), J2.4 (Pin_4), J3.4 (Pin_4), M1.2 (3V3), M2.8 (3.3V), R10.1, R9.1, U1.16 (3V3); no longer R7.2, R8.2
- net +5V: now also C1.1, C10.1, C2.1, J5.2 (Pin_2), M1.15 (5V), M1.16 (5V)
- net GND: now also C1.2, C10.2, C2.2, C3.2, C7.2, J1.5 (Pin_5), J2.5 (Pin_5), J3.5 (Pin_5), M1.1 (GND), M1.17 (GND), M1.30 (GND), M2.15 (GND), M2.2 (GND), M2.7 (GND), M3.5 (0V), U1.17 (GND), U1.18 (GND), U4.2, U5.3, U6.3, U7.2, U8.2
- net STM_RX: no longer D5.1 (K)
- net I2C1_SCL: no longer names the net of R7.1
- net I2C1_SCL: now also U4.1
- net I2C1_SDA: no longer names the net of R8.1
- net I2C1_SDA: now also Q1.2 (B), U4.4, U9.2 (TRIG)
- net PA2 renamed LED3
- net LED3: now also M1.23 (D22), U1.4 (PB15)
- net PA3 renamed LED1
- net LED1: now also M1.8 (D0), U1.20 (PB9)
- net PA4 renamed LED4
- net LED4: now also M1.25 (D15), U1.5 (PA8)
- net PA5 renamed LED2
- net LED2: now also M1.9 (D1), U1.19 (PB8)
- net STM_TX renamed UART_AT_TX
- net UART_AT_TX: now also M1.26 (RX), U1.6 (PA9)
- new net: R11.1, U7.1
- new net: C11.1, R13.1, R14.1, U9.6 (THRES), U9.7 (DISCH)
- new net: R12.1, U8.1
- new net: Q1.3 (E), R13.2
- new net: J5.1 (Pin_1), M3.6 (+Vo)
- new net HI_GND: C11.2, C12.2, J6.2, J7.2, J7.4, J9.2, M3.2 (GND), Q1.1 (C), U4.3, U5.2, U6.2, U7.3, U8.3, U9.1 (GND)
- new net IN1_3V3: M1.24 (D23), R9.2, U1.31 (PB0), U5.4
- new net IN1_DRY1: J8.1, R15.2
- new net IN1_DRY2: J8.2, U5.1
- new net IN2_3V3: M1.10 (D8), R10.2, U1.15 (PB7), U6.4
- new net IN2_DRY1: J8.3, R16.2
- new net IN2_DRY2: J8.4, U6.1
- new net LM555_ON_PULSE: M1.22 (D21), R7.2, U1.2 (PB13)
- new net LR1121_BUSY: M1.19 (D18), M2.9 (BUSY), U1.24 (PA1)
- new net LR1121_IRQ: M1.28 (D3), M2.3 (DIO9), U1.10 (PA15)
- new net LR1121_RESET: M1.12 (D11), M2.10 (RESET), U1.27 (PA4)
- new net LR1121_SSEL: M1.11 (D10), M2.14 (CS), U1.11 (PB3)
- new net MISO: J1.1 (Pin_1), J2.1 (Pin_1), J3.1 (Pin_1), M1.29 (D2), M2.11 (MISO), U1.12 (PB4)
- new net MOSI: M1.7 (D7), M2.12 (MOSI), U1.13 (PB5)
- new net OUT1_3V3: R11.2, U1.3 (PB14)
- new net OUT1_OC: J7.1, U7.4
- new net OUT2_3V3: M1.18 (D9), R12.2, U1.14 (PB6)
- new net OUT2_OC: J7.3, U8.4
- new net PULSE_DETECTOR_OUT: J9.1, U9.3 (OUT)
- new net SCLK: J1.3 (Pin_3), J2.3 (Pin_3), J3.3 (Pin_3), M1.6 (D6), M2.13 (SCLK), U1.28 (PA5)
- new net TEMP1_SSEL: J2.2 (Pin_2), M1.20 (D19), U1.26 (PA3)
- new net TEMP2_SSEL: J1.2 (Pin_2), M1.21 (D20), U1.25 (PA2)
- new net TEMP3_SSEL: J3.2 (Pin_2), M1.5 (D5), U1.34 (PB11)
- new net UART_AT_RX: D5.1 (K), M1.27 (TX), U1.7 (PA10)
- no-connect marks 26 -> 18
Other:
- note added: "Domínio 12V"
- note added: "Termopares"
- note removed: "4 - Interface"
- note removed: "6 - BMP180"
- note removed: "7 - LM35"
- note removed: "Blackpill"
- note removed: "GND on pin 40 was left unconnected to ensure blackpill compatibility"
- note removed: "LED1"
- note removed: "LED2"
- note removed: "LED3"
- note removed: "LED4"
- note removed: "PA0"
- note removed: "PA1"
- note removed: "PA2"
- note removed: "PA3"
- note removed: "PA4"
- note removed: "PA6"
- note removed: "PA7"
- note removed: "PA8"
- note removed: "PB12"
- note removed: "PB13"
- note removed: "PB2"
- note removed: "PB3"
- note removed: "PB4"
- note removed: "PB5"
- note removed: "PB6"
- note removed: "PB7"
- note removed: "PB8"
- note removed: "PB9"
- title: Bluepill + Radioenge AT interface -> Blackpill/ESP32C6 + Radioenge AT interface + LR1121
- moved on the sheet: C4, C5, C6, C8, C9, D1, D2, D3, D4, D5, D6, D7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

Commit message: add footprints, wip
Co-Authored-By: Claude Sonnet 5 <noreply@anthropic.com>
Parts:
- M1: footprint (none) -> LabSC:ESP32C6-Minimal
- M2: footprint (none) -> LabSC:Waveshare-LR1121
- M3: footprint (none) -> LabSC:A1205S-2W
Changed lines of the file:
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@@
 			)
 		)
-		(property "Footprint" ""
+		(property "Footprint" "LabSC:ESP32C6-Minimal"
 			(at 35.56 116.84 0)
 			(hide yes)
@@
 		(in_pos_files yes)
 		(dnp no)
-		(fields_autoplaced yes)
 		(property "Reference" "M2"
 			(at 218.0433 95.25 0)
@@
 			)
 		)
-		(property "Footprint" ""
-			(at 204.47 97.79 0)
-			(hide yes)
+		(property "Footprint" "LabSC:Waveshare-LR1121"
+			(at 197.866 95.758 0)
 			(show_name no)
 			(do_not_autoplace no)
@@
 			)
 		)
-		(property "Footprint" ""
+		(property "Footprint" "LabSC:A1205S-2W"
 			(at 364.49 31.75 0)
 			(hide yes)

Commit message: WIP: schematic/PCB progress, screw terminals, ESP32-C6 reference
Design work in progress on the LoRa carrier:
  - schematic and PCB updates
  - HANDSON KF301-2P / KF301-4P screw terminal footprints
  - Custom_Symbols.kicad_sym
  - Connector.kicad_sym additions, fp-lib-table / sym-lib-table updates
  - Waveshare-LR1121 footprint tweak
  - nanoESP32C6.pdf: module reference schematic. Confirms the onboard LED is
    an addressable RGB (WS2812-type) driven from GPIO8, not a plain GPIO LED.

Bumps the Kicad-STM32 submodule to 244753d, which adds the two BlackPill
symbols that were sitting untracked in the submodule working tree.

Co-Authored-By: Claude Opus 4.8 <noreply@anthropic.com>
Parts:
- removed J3: Conn_01x05, symbol Connector_Generic:Conn_01x05
- removed J6, J9: (no value), symbol Connector:Screw01x02
- removed J7, J8: (no value), symbol Connector:Screw01x04
- removed U1: YAAJ_BlackPill, Footprints:YAAJ_WeAct_BlackPill_2, symbol YAAJ_BlackPill:YAAJ_BlackPill
- added J10, J11: Screw_Terminal_01x04, KF301-2P:HANDSON_KF301-4P, symbol Connector:Screw_Terminal_01x04
- added J7, J8: Screw_Terminal_01x02, KF301-2P:HANDSON_KF301-2P, symbol Connector:Screw_Terminal_01x02
- added U10: YAAJ_WeAct_BlackPill_Part_Like, Footprints:YAAJ_WeAct_BlackPill_2, symbol YAAJ_WeAct_BlackPill_Part_Like:YAAJ_WeAct_BlackPill_Part_Like
- C10: footprint Capacitor_SMD:CP_Elec_5x3 -> Capacitor_THT:CP_Radial_D5.0mm_P2.50mm
- C12: footprint Capacitor_SMD:CP_Elec_4x3 -> Capacitor_THT:CP_Radial_D5.0mm_P2.50mm
- J1, J2: footprint (none) -> Connector_PinHeader_2.54mm:PinHeader_1x05_P2.54mm_Horizontal
- J5: footprint (none) -> Connector_PinHeader_2.54mm:PinHeader_1x02_P2.54mm_Vertical
Connections:
- net TEMP3_SSEL is gone; now on net LR1121_SSEL: M1.5 (D5)
- net +12V: now also J7.1 (Pin_1)
- net +3V3: now also U10.20 (3V3), U10.38 (3V3)
- net +5V: now also U10.18 (5V), U10.40 (5V)
- net GND: now also U10.19 (GND), U10.39 (GND)
- net HI_GND: now also J10.2 (Pin_2), J10.4 (Pin_4), J7.2 (Pin_2), J8.2 (Pin_2)
- net IN1_3V3: now also U10.33 (PA7)
- net IN1_DRY1: now also J11.1 (Pin_1)
- net IN1_DRY2: now also J11.2 (Pin_2)
- net IN2_3V3: now also M1.20 (D19), U10.30 (PA4); no longer M1.10 (D8)
- net IN2_DRY1: now also J11.3 (Pin_3)
- net IN2_DRY2: now also J11.4 (Pin_4)
- net LED1: now also U10.1 (PB12); no longer M1.8 (D0)
- net LED2: now also U10.2 (PB13); no longer M1.9 (D1)
- net LED3: now also U10.3 (PB14); no longer M1.23 (D22)
- net LED4: now also U10.4 (PB15); no longer M1.25 (D15)
- net LM555_ON_PULSE: now also U10.35 (PB1)
- net LR1121_BUSY: now also M1.11 (D10), U10.16 (PB8); no longer M1.19 (D18)
- net LR1121_IRQ: now also M1.12 (D11), U10.17 (PB9); no longer M1.28 (D3)
- net LR1121_RESET: now also M1.9 (D1), U10.14 (PB6); no longer M1.12 (D11)
- net LR1121_SSEL: now also U10.10 (PA15); no longer M1.11 (D10)
- net MISO: now also M1.7 (D7), U10.12 (PB4); no longer M1.29 (D2)
- net MOSI: now also M1.8 (D0), U10.13 (PB5); no longer M1.7 (D7)
- net OUT1_3V3: now also M1.21 (D20), U10.37 (PB10)
- net OUT1_OC: now also J10.1 (Pin_1)
- net OUT2_3V3: now also M1.25 (D15), U10.32 (PA6); no longer M1.18 (D9)
- net OUT2_OC: now also J10.3 (Pin_3)
- net PULSE_DETECTOR_OUT: now also J8.1 (Pin_1)
- net SCLK: now also U10.11 (PB3)
- net TEMP1_SSEL: now also M1.4 (D4), U10.9 (PA12); no longer M1.20 (D19)
- net TEMP2_SSEL: now also U10.34 (PB0); no longer M1.21 (D20)
- net UART_AT_RX: now also M1.26 (RX), U10.29 (PA3); no longer M1.27 (TX)
- net UART_AT_TX: now also M1.27 (TX), U10.28 (PA2); no longer M1.26 (RX)
- no-connect marks 18 -> 35
Other:
- moved on the sheet: C1, C2, C3, C4, C5, C6, J2
