File: lora-bluepill-sch.kicad_sch (KiCad schematic)
At the start: 62 parts, among them J1 Conn_01x05, J10 Screw_Terminal_01x04, J11 Screw_Terminal_01x04, J2 Conn_01x05, J4 Conn_01x04_Male, J5 Conn_01x02, J7 Screw_Terminal_01x02, J8 Screw_Terminal_01x02, Q1 BC558, U10 YAAJ_WeAct_BlackPill_Part_Like, U2 FTDI_Breakout, U3 RadioEnge_LoRaWAN, U4 PC817, U5 PC817, U6 PC817, U7 PC817, U8 PC817, U9 NE555P

Commit message: placement evolution
Parts:
- added R17: 1K, Resistor_THT:R_Axial_DIN0204_L3.6mm_D1.6mm_P7.62mm_Horizontal, symbol Device:R
Connections:
- net STM_RX is gone; now on net UART_AT_RX: U3.3 (AT_TX)
- net +3V3: now also R17.1
- net IN1_3V3: now also M1.28 (D3); no longer M1.24 (D23)
- net IN2_3V3: now also M1.26 (RX), U10.31 (PA5); no longer M1.20 (D19), U10.30 (PA4)
- net LM555_ON_PULSE: now also U10.27 (PA1); no longer U10.35 (PB1)
- net OUT1_3V3: now also U10.26 (PA0); no longer U10.37 (PB10)
- net OUT2_3V3: now also U10.30 (PA4), R17.2; no longer U10.32 (PA6)
- net TEMP2_SSEL: now also M1.29 (D2)
- net UART_AT_RX: now also M1.24 (D23); no longer M1.26 (RX)
- net UART_AT_TX: now also M1.23 (D22); no longer M1.27 (TX)
- net AT_RX: no longer names the net of D7.2 (A), D8.2 (A), R6.2, U3.2 (AT_RX)
- no-connect marks 35 -> 34
Other:
- note added: "D15 needs a pullup to proper JTAG config"

Commit message: board finished, but not checked
Parts:
- removed C7, C8: 100n, Capacitor_THT:C_Disc_D6.0mm_W4.4mm_P5.00mm, symbol Device:C
- removed J4: Conn_01x04_Male, Connector_PinSocket_2.54mm:PinSocket_1x04_P2.54mm_Vertical, symbol Connector:Conn_01x04_Male
- added C13, C14, C15, C16: 100n, Capacitor_THT:C_Disc_D6.0mm_W4.4mm_P5.00mm, symbol Device:C
- added D10: 5V, Diode_THT:D_DO-35_SOD27_P7.62mm_Horizontal, symbol Diode:Zener
- added R18: 100, Resistor_THT:R_Axial_DIN0204_L3.6mm_D1.6mm_P7.62mm_Horizontal, symbol Device:R
Connections:
- net +12V: now also U9.4 (~{RST}), C15.1, C16.1
- net +3V3: now also C14.1
- net +5V: now also C13.1, D10.1 (K)
- net GND: now also C13.2, C14.2, R18.2
- net HI_GND: now also J10.1 (Pin_1), J10.3 (Pin_3), C15.2, C16.2; no longer J10.2 (Pin_2), J10.4 (Pin_4)
- net IN2_3V3: now also M1.24 (D23); no longer M1.26 (RX)
- net OUT1_OC: now also J10.4 (Pin_4); no longer J10.1 (Pin_1)
- net OUT2_OC: now also J10.2 (Pin_2); no longer J10.3 (Pin_3)
- net TEMP1_SSEL: now also U10.5 (PA8); no longer U10.9 (PA12)
- net UART_AT_RX: now also M1.26 (RX); no longer M1.24 (D23)
- net UART_AT_TX: now also M1.27 (TX); no longer M1.23 (D22)
- net EXP_C6_TX: now reaches M1.18 (D9)
- net EXP_C6_SCL: now reaches M1.19 (D18)
- net EXP_C6_SDA: now reaches M1.20 (D19)
- net FTDI_5V: no longer names the net of U2.4 (VCC)
- net FTDI_RX: no longer names the net of D4.2 (A), D5.2 (A), R3.2, U2.2 (RX)
- new net: D10.2 (A), R18.1
- new net EXP_C6_RX: M1.23 (D22)
- no-connect marks 34 -> 32
Other:
- moved on the sheet: C10, J5, M3
